File: pcb/tank_controller.kicad_pcb (KiCad board)
At the start: 2 copper layers, 100 x 98 mm, 26 parts, among them J1 MAINS IN, J2 SELECTOR S1, J3 KM COIL, J4 LAMP H1, J5 SENSOR, J6 ESP32 3V3 side, J7 ESP32 VIN side, K1 G5NB-1A-E 5VDC, Q1 BC547

Commit message: Rev 1.1: polarity marks that survive the silk clean-up, in-stock BOM parts.
The October 2026 boards came with Q1 backwards: pull_silk() had stripped the
TO-92 outline, leaving only a straight line. Copper is unchanged.
Other:
- board text added: "B"
- board text added: "C"
- board text added: "E"
- board text added: "REV 1.1"
